File: disp.kicad_sch (KiCad schematic)
At the start: 15 parts, among them J5 Conn_01x07_Socket, J6 Conn_01x07_Socket, J7 Conn_01x07_Socket, J8 Conn_01x07_Socket, U6 MAX7221CWGT+, U7 MAX7221CWGT

Commit message: Updated BOM, created fab outputs
Parts:
- J5, J6, J7, J8: Mfr (none) -> Adam Tech; Mfr P/N (none) -> PH1-07-UA; Supplier 1 (none) -> Digikey; Supplier 1 P/N (none) -> 2057-PH1-07-UA-ND; Supplier 1 Price @ Qty (none) -> 0.14000; Supplier 1 Unit Price (none) -> 0.14000
- R33, R34, R35, R38, R39, R40: Supplier 1 P/N (none) -> 311-0.0GRTR-ND; Supplier 1 Price @ Qty (none) -> 0.00900; Supplier 1 Unit Price (none) -> 0.10
- R36: Supplier 1 P/N (none) -> RNCP0603FTD10K0CT-ND; Supplier 1 Price @ Qty (none) -> 0.10; Supplier 1 Unit Price (none) -> 0.10
- R37, R41: Supplier_1 P/N (none) -> 118-CR0603-FX-9531ELFTR-ND; Supplier_1 Price @ Qty (none) -> 0.10000; Supplier_1 Unit Price (none) -> 0.10000
- U6, U7: Mfr P/N MAX7219CWG+T -> MAX7221CWG+T; Supplier 1 P/N MAX7219CWG+TTR-ND -> MAX7221CWG+CT-ND; Supplier 1 Price @ Qty 17.90000 -> 17.31; Supplier 1 Unit Price 17.90000 -> 17.31; Supplier_1 P/N (none) -> MAX7219CWG+TTR-ND; Supplier_1 Price @ Qty (none) -> 17.90000; Supplier_1 Unit Price (none) -> 17.90000
