File: light.kicad_sch (KiCad schematic)
At the start: 3 parts, among them J4 Conn_01x05

Commit message: Updated BOM, created fab outputs
Parts:
- J4: Supplier_1 P/N (none) -> S6103-ND; Supplier_1 Price @ Qty (none) -> 0.57000; Supplier_1 Unit Price (none) -> 0.57000
- R31, R32: Supplier 1 P/N (none) -> 311-0.0GRTR-ND; Supplier 1 Price @ Qty (none) -> 0.00900; Supplier 1 Unit Price (none) -> 0.10
Changed lines of the file:
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@@
 			)
 		)
-		(property "Supplier 1 P/N" ""
-			(at 78.74 85.09 0)
-			(effects
-				(font
-					(size 1.27 1.27)
-				)
-				(hide yes)
-			)
-		)
-		(property "Supplier 1 Unit Price" ""
-			(at 78.74 85.09 0)
-			(effects
-				(font
-					(size 1.27 1.27)
-				)
-				(hide yes)
-			)
-		)
-		(property "Supplier 1 Price @ Qty" ""
+		(property "Supplier 1 P/N" "311-0.0GRTR-ND"
+			(at 78.74 85.09 0)
+			(effects
+				(font
+					(size 1.27 1.27)
+				)
+				(hide yes)
+			)
+		)
+		(property "Supplier 1 Unit Price" "0.10"
+			(at 78.74 85.09 0)
+			(effects
+				(font
+					(size 1.27 1.27)
+				)
+				(hide yes)
+			)
+		)
+		(property "Supplier 1 Price @ Qty" "0.00900"
 			(at 78.74 85.09 0)
 			(effects
@@
 			)
 		)
-		(property "Supplier 1 P/N" ""
-			(at 78.74 87.63 0)
-			(effects
-				(font
-					(size 1.27 1.27)
-				)
-				(hide yes)
-			)
-		)
-		(property "Supplier 1 Unit Price" ""
-			(at 78.74 87.63 0)
-			(effects
-				(font
-					(size 1.27 1.27)
-				)
-				(hide yes)
-			)
-		)
-		(property "Supplier 1 Price @ Qty" ""
+		(property "Supplier 1 P/N" "311-0.0GRTR-ND"
+			(at 78.74 87.63 0)
+			(effects
+				(font
+					(size 1.27 1.27)
+				)
+				(hide yes)
+			)
+		)
+		(property "Supplier 1 Unit Price" "0.10"
+			(at 78.74 87.63 0)
+			(effects
+				(font
+					(size 1.27 1.27)
+				)
+				(hide yes)
+			)
+		)
+		(property "Supplier 1 Price @ Qty" "0.00900"
 			(at 78.74 87.63 0)
 			(effects
@@
 			(at 96.52 82.55 0)
 			(effects
+				(font
+					(size 1.27 1.27)
+				)
+				(hide yes)
+			)
+		)
+		(property "Supplier_1 P/N" "S6103-ND"
+			(at 96.52 82.55 0)
+			(effects
+				(font
+					(size 1.27 1.27)
+				)
+				(hide yes)
+			)
+		)
+		(property "Supplier_1 Price @ Qty" "0.57000"
+			(at 96.52 82.55 0)
+			(effects
+				(font
+					(size 1.27 1.27)
+				)
+				(hide yes)
+			)
+		)
+		(property "Supplier_1 Unit Price" "0.57000"
+			(at 96.52 82.55 0)
+			(effects
