File: mcu.kicad_sch (KiCad schematic)
At the start: 13 parts, among them X3 32.768 kHz

Commit message: Updated BOM, created fab outputs
Parts:
- C15, C16: Supplier 1 P/N (none) -> 399-C0603C220K4GAC7867CT-ND; Supplier 1 Price @ Qty (none) -> 0.10; Supplier 1 Unit Price (none) -> 0.10
- LED1: Supplier 1 P/N (none) -> 2686; Supplier 1 Price @ Qty (none) -> 0.495; Supplier 1 Unit Price (none) -> 0.495
- R11, R12: Supplier 1 P/N (none) -> CR0603-FX-1003ELFTR-ND; Supplier 1 Price @ Qty (none) -> 0.10000; Supplier 1 Unit Price (none) -> 0.10
- R13: Supplier 1 P/N (none) -> A129540CT-ND; Supplier 1 Price @ Qty (none) -> 0.10; Supplier 1 Unit Price (none) -> 0.10
- R14: Supplier 1 P/N (none) -> RNCP0603FTD10K0CT-ND; Supplier 1 Price @ Qty (none) -> 0.10; Supplier 1 Unit Price (none) -> 0.10
- U$1: Supplier 1 (none) -> Digikey; Supplier 1 P/N (none) -> ATSAMD51J19A-AUTCT-ND; Supplier 1 Price @ Qty (none) -> 5.68; Supplier 1 Unit Price (none) -> 5.68
- X3: Supplier 1 (none) -> Digikey; Supplier 1 P/N (none) -> 644-STDMUA17-32.768KCT-ND; Supplier 1 Price @ Qty (none) -> 1.02000; Supplier 1 Unit Price (none) -> 1.02000
Changed lines of the file:
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@@
 			)
 		)
+		(property "Supplier 1 P/N" "644-STDMUA17-32.768KCT-ND"
+			(at 149.86 40.64 0)
+			(effects
+				(font
+					(size 1.27 1.27)
+				)
+				(hide yes)
+			)
+		)
+		(property "Supplier 1 Price @ Qty" "1.02000"
+			(at 149.86 40.64 0)
+			(effects
+				(font
+					(size 1.27 1.27)
+				)
+				(hide yes)
+			)
+		)
+		(property "Supplier 1 Unit Price" "1.02000"
+			(at 149.86 40.64 0)
+			(effects
+				(font
+					(size 1.27 1.27)
+				)
+				(hide yes)
+			)
+		)
+		(property "Supplier 1" "Digikey"
+			(at 149.86 40.64 0)
+			(effects
+				(font
+					(size 1.27 1.27)
+				)
+				(hide yes)
+			)
+		)
 		(pin "P$1"
 		)
@@
 			)
 		)
+		(property "Supplier 1 P/N" "399-C0603C220K4GAC7867CT-ND"
+			(at 139.7 35.56 0)
+			(effects
+				(font
+					(size 1.27 1.27)
+				)
+				(hide yes)
+			)
+		)
+		(property "Supplier 1 Price @ Qty" "0.10"
+			(at 139.7 35.56 0)
+			(effects
+				(font
+					(size 1.27 1.27)
+				)
+				(hide yes)
+			)
+		)
+		(property "Supplier 1 Unit Price" "0.10"
+			(at 139.7 35.56 0)
+			(effects
+				(font
+					(size 1.27 1.27)
+				)
+				(hide yes)
+			)
+		)
 		(pin "1"
 		)
@@
 			)
 		)
+		(property "Supplier 1 P/N" "CR0603-FX-1003ELFTR-ND"
+			(at 118.11 107.95 0)
+			(effects
+				(font
+					(size 1.27 1.27)
+				)
+				(hide yes)
+			)
+		)
+		(property "Supplier 1 Price @ Qty" "0.10000"
+			(at 118.11 107.95 0)
+			(effects
+				(font
+					(size 1.27 1.27)
+				)
+				(hide yes)
+			)
+		)
+		(property "Supplier 1 Unit Price" "0.10"
+			(at 118.11 107.95 0)
+			(effects
+				(font
+					(size 1.27 1.27)
+				)
+				(hide yes)
+			)
+		)
 		(pin "1"
 		)
@@
 			)
 		)
+		(property "Supplier 1 P/N" "ATSAMD51J19A-AUTCT-ND"
+			(at 209.55 121.92 0)
+			(effects
+				(font
+					(size 1.27 1.27)
+				)
+				(hide yes)
+			)
+		)
+		(property "Supplier 1 Price @ Qty" "5.68"
+			(at 209.55 121.92 0)
+			(effects
+				(font
+					(size 1.27 1.27)
+				)
+				(hide yes)
+			)
+		)
+		(property "Supplier 1 Unit Price" "5.68"
+			(at 209.55 121.92 0)
+			(effects
+				(font
+					(size 1.27 1.27)
+				)
+				(hide yes)
+			)
+		)
+		(property "Supplier 1" "Digikey"
+			(at 209.55 121.92 0)
+			(effects
+				(font
+					(size 1.27 1.27)
+				)
+				(hide yes)
+			)
+		)
 		(pin "1"
 		)
@@
 			)
 		)
-		(property "Supplier 1" ""
+		(property "Supplier 1" "Digikey"
 			(at 190.5 66.04 0)
 			(effects
@@
 			)
 		)
-		(property "Supplier 1 P/N" ""
+		(property "Supplier 1 P/N" "ATSAMD51J19A-AUTCT-ND"
 			(at 190.5 66.04 0)
 			(effects
@@
 			)
 		)
-		(property "Supplier 1 Unit Price" ""
+		(property "Supplier 1 Unit Price" "5.68"
 			(at 190.5 66.04 0)
 			(effects
@@
 			)
 		)
-		(property "Supplier 1 Price @ Qty" ""
+		(property "Supplier 1 Price @ Qty" "5.68"
 			(at 190.5 66.04 0)
 			(effects
@@
 			)
 		)
+		(property "Supplier 1 P/N" "2686"
+			(at 91.44 132.08 0)
+			(effects
+				(font
+					(size 1.27 1.27)
+				)
+				(hide yes)
+			)
+		)
+		(property "Supplier 1 Price @ Qty" "0.495"
+			(at 91.44 132.08 0)
+			(effects
+				(font
+					(size 1.27 1.27)
+				)
+				(hide yes)
+			)
+		)
+		(property "Supplier 1 Unit Price" "0.495"
+			(at 91.44 132.08 0)
+			(effects
+				(font
+					(size 1.27 1.27)
+				)
+				(hide yes)
+			)
+		)
 		(pin "1"
 		)
@@
 			)
 		)
-		(property "Supplier 1 P/N" ""
+		(property "Supplier 1 P/N" "A129540CT-ND"
 			(at 293.37 66.04 0)
 			(effects
@@
 			)
 		)
-		(property "Supplier 1 Unit Price" ""
+		(property "Supplier 1 Unit Price" "0.10"
 			(at 293.37 66.04 0)
 			(effects
@@
 			)
 		)
-		(property "Supplier 1 Price @ Qty" ""
+		(property "Supplier 1 Price @ Qty" "0.10"
 			(at 293.37 66.04 0)
 			(effects
@@
 			)
 		)
-		(property "Supplier 1 P/N" ""
+		(property "Supplier 1 P/N" "RNCP0603FTD10K0CT-ND"
 			(at 313.69 73.66 0)
 			(effects
@@
 			)
 		)
-		(property "Supplier 1 Unit Price" ""
+		(property "Supplier 1 Unit Price" "0.10"
 			(at 313.69 73.66 0)
 			(effects
@@
 			)
 		)
-		(property "Supplier 1 Price @ Qty" ""
+		(property "Supplier 1 Price @ Qty" "0.10"
 			(at 313.69 73.66 0)
 			(effects
@@
 			)
 		)
+		(property "Supplier 1 P/N" "CR0603-FX-1003ELFTR-ND"
+			(at 118.11 115.57 0)
+			(effects
+				(font
+					(size 1.27 1.27)
+				)
+				(hide yes)
+			)
+		)
+		(property "Supplier 1 Price @ Qty" "0.10000"
+			(at 118.11 115.57 0)
+			(effects
+				(font
+					(size 1.27 1.27)
+				)
+				(hide yes)
+			)
+		)
+		(property "Supplier 1 Unit Price" "0.10"
+			(at 118.11 115.57 0)
+			(effects
+				(font
+					(size 1.27 1.27)
+				)
+				(hide yes)
+			)
+		)
 		(pin "1"
 		)
@@
 			(at 139.7 45.72 0)
 			(effects
+				(font
+					(size 1.27 1.27)
+				)
+				(hide yes)
+			)
+		)
+		(property "Supplier 1 P/N" "399-C0603C220K4GAC7867CT-ND"
+			(at 139.7 45.72 0)
+			(effects
+				(font
+					(size 1.27 1.27)
+				)
+				(hide yes)
+			)
+		)
+		(property "Supplier 1 Price @ Qty" "0.10"
+			(at 139.7 45.72 0)
+			(effects
+				(font
+					(size 1.27 1.27)
+				)
+				(hide yes)
+			)
+		)
+		(property "Supplier 1 Unit Price" "0.10"
+			(at 139.7 45.72 0)
+			(effects
