File: microsd.kicad_sch (KiCad schematic)
At the start: 9 parts, among them J2 MEM2075-00-140-01-A

Commit message: Updated BOM, created fab outputs
Parts:
- J2: Mfr (none) -> GCT; Mfr P/N (none) -> MEM2075-00-140-01-A; Supplier 1 Price @ Qty (none) -> 2.45000; Supplier 1 Unit Price (none) -> 2.45000; Supplier_1 P/N (none) -> 2073-MEM2075-00-140-01-ATR-ND; Supplier_1 Price @ Qty (none) -> 2073-MEM2075-00-140-01-ATR-ND; Supplier_1 Unit Price (none) -> 2073-MEM2075-00-140-01-ATR-ND
- R15, R16, R17, R18: Supplier 1 P/N (none) -> 311-0.0GRTR-ND; Supplier 1 Price @ Qty (none) -> 0.00900; Supplier 1 Unit Price (none) -> 0.10
- R19, R20, R21, R22: Supplier 1 P/N (none) -> CR0603-FX-4702ELFTR-ND; Supplier 1 Price @ Qty (none) -> 0.10; Supplier 1 Unit Price (none) -> 0.10
Changed lines of the file:
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@@
 			)
 		)
-		(property "Supplier 1 P/N" ""
+		(property "Supplier 1 P/N" "311-0.0GRTR-ND"
 			(at 85.09 95.25 0)
 			(effects
@@
 			)
 		)
-		(property "Supplier 1 Unit Price" ""
+		(property "Supplier 1 Unit Price" "0.10"
 			(at 85.09 95.25 0)
 			(effects
@@
 			)
 		)
-		(property "Supplier 1 Price @ Qty" ""
+		(property "Supplier 1 Price @ Qty" "0.00900"
 			(at 85.09 95.25 0)
 			(effects
@@
 			)
 		)
-		(property "Supplier 1 P/N" ""
+		(property "Supplier 1 P/N" "CR0603-FX-4702ELFTR-ND"
 			(at 100.33 78.74 0)
 			(effects
@@
 			)
 		)
-		(property "Supplier 1 Unit Price" ""
+		(property "Supplier 1 Unit Price" "0.10"
 			(at 100.33 78.74 0)
 			(effects
@@
 			)
 		)
-		(property "Supplier 1 Price @ Qty" ""
+		(property "Supplier 1 Price @ Qty" "0.10"
 			(at 100.33 78.74 0)
 			(effects
@@
 			)
 		)
+		(property "Supplier_1 P/N" "2073-MEM2075-00-140-01-ATR-ND"
+			(at 139.7 95.25 0)
+			(effects
+				(font
+					(size 1.27 1.27)
+				)
+				(hide yes)
+			)
+		)
+		(property "Supplier_1 Price @ Qty" "2073-MEM2075-00-140-01-ATR-ND"
+			(at 139.7 95.25 0)
+			(effects
+				(font
+					(size 1.27 1.27)
+				)
+				(hide yes)
+			)
+		)
+		(property "Supplier_1 Unit Price" "2073-MEM2075-00-140-01-ATR-ND"
+			(at 139.7 95.25 0)
+			(effects
+				(font
+					(size 1.27 1.27)
+				)
+				(hide yes)
+			)
+		)
+		(property "Mfr" "GCT"
+			(at 139.7 95.25 0)
+			(effects
+				(font
+					(size 1.27 1.27)
+				)
+				(hide yes)
+			)
+		)
+		(property "Mfr P/N" "MEM2075-00-140-01-A"
+			(at 139.7 95.25 0)
+			(effects
+				(font
+					(size 1.27 1.27)
+				)
+				(hide yes)
+			)
+		)
+		(property "Supplier 1 Price @ Qty" "2.45000"
+			(at 139.7 95.25 0)
+			(effects
+				(font
+					(size 1.27 1.27)
+				)
+				(hide yes)
+			)
+		)
+		(property "Supplier 1 Unit Price" "2.45000"
+			(at 139.7 95.25 0)
+			(effects
+				(font
+					(size 1.27 1.27)
+				)
+				(hide yes)
+			)
+		)
 		(pin "SH1"
 		)
@@
 			)
 		)
-		(property "Supplier 1 P/N" ""
+		(property "Supplier 1 P/N" "311-0.0GRTR-ND"
 			(at 85.09 87.63 0)
 			(effects
@@
 			)
 		)
-		(property "Supplier 1 Unit Price" ""
+		(property "Supplier 1 Unit Price" "0.10"
 			(at 85.09 87.63 0)
 			(effects
@@
 			)
 		)
-		(property "Supplier 1 Price @ Qty" ""
+		(property "Supplier 1 Price @ Qty" "0.00900"
 			(at 85.09 87.63 0)
 			(effects
@@
 			)
 		)
-		(property "Supplier 1 P/N" ""
+		(property "Supplier 1 P/N" "311-0.0GRTR-ND"
 			(at 85.09 90.17 0)
 			(effects
@@
 			)
 		)
-		(property "Supplier 1 Unit Price" ""
+		(property "Supplier 1 Unit Price" "0.10"
 			(at 85.09 90.17 0)
 			(effects
@@
 			)
 		)
-		(property "Supplier 1 Price @ Qty" ""
+		(property "Supplier 1 Price @ Qty" "0.00900"
 			(at 85.09 90.17 0)
 			(effects
@@
 			)
 		)
-		(property "Supplier 1 P/N" ""
+		(property "Supplier 1 P/N" "311-0.0GRTR-ND"
 			(at 85.09 92.71 0)
 			(effects
@@
 			)
 		)
-		(property "Supplier 1 Unit Price" ""
+		(property "Supplier 1 Unit Price" "0.10"
 			(at 85.09 92.71 0)
 			(effects
@@
 			)
 		)
-		(property "Supplier 1 Price @ Qty" ""
+		(property "Supplier 1 Price @ Qty" "0.00900"
 			(at 85.09 92.71 0)
 			(effects
@@
 			)
 		)
-		(property "Supplier 1 P/N" ""
+		(property "Supplier 1 P/N" "CR0603-FX-4702ELFTR-ND"
 			(at 91.44 78.74 0)
 			(effects
@@
 			)
 		)
-		(property "Supplier 1 Unit Price" ""
+		(property "Supplier 1 Unit Price" "0.10"
 			(at 91.44 78.74 0)
 			(effects
@@
 			)
 		)
-		(property "Supplier 1 Price @ Qty" ""
+		(property "Supplier 1 Price @ Qty" "0.10"
 			(at 91.44 78.74 0)
 			(effects
@@
 			)
 		)
-		(property "Supplier 1 P/N" ""
+		(property "Supplier 1 P/N" "CR0603-FX-4702ELFTR-ND"
 			(at 115.57 78.74 0)
 			(effects
@@
 			)
 		)
-		(property "Supplier 1 Unit Price" ""
+		(property "Supplier 1 Unit Price" "0.10"
 			(at 115.57 78.74 0)
 			(effects
@@
 			)
 		)
-		(property "Supplier 1 Price @ Qty" ""
+		(property "Supplier 1 Price @ Qty" "0.10"
 			(at 115.57 78.74 0)
 			(effects
@@
 			)
 		)
-		(property "Supplier 1 P/N" ""
+		(property "Supplier 1 P/N" "CR0603-FX-4702ELFTR-ND"
 			(at 107.95 78.74 0)
 			(effects
@@
 			)
 		)
-		(property "Supplier 1 Unit Price" ""
+		(property "Supplier 1 Unit Price" "0.10"
 			(at 107.95 78.74 0)
 			(effects
@@
 			)
 		)
-		(property "Supplier 1 Price @ Qty" ""
+		(property "Supplier 1 Price @ Qty" "0.10"
 			(at 107.95 78.74 0)
 			(effects
