File: onoff.kicad_sch (KiCad schematic)
At the start: 9 parts, among them Q2 MMBT2222A-7-F, U3 AT42QT1011-TSHR

Commit message: Updated BOM, created fab outputs
Parts:
- C13, C14: Supplier_1 P/N (none) -> 399-C0402C103K3REC7411TR-ND; Supplier_1 Price @ Qty (none) -> 0.10000; Supplier_1 Unit Price (none) -> 0.10000
- D2: Supplier_1 P/N (none) -> 732-4980-2-ND; Supplier_1 Price @ Qty (none) -> 0.15000; Supplier_1 Unit Price (none) -> 0.15000
- Q2: Supplier_1 P/N (none) -> MMBT2222A-FDITR-ND; Supplier_1 Price @ Qty (none) -> 0.10000; Supplier_1 Unit Price (none) -> 0.10000
- R7: Supplier 1 P/N (none) -> A129540CT-ND; Supplier 1 Price @ Qty (none) -> 0.10; Supplier 1 Unit Price (none) -> 0.10
- R8: Supplier_1 P/N (none) -> 118-CR0603-FX-2000ELFTR-ND; Supplier_1 Price @ Qty (none) -> 0.10000; Supplier_1 Unit Price (none) -> 0.10000
- R9: Supplier 1 P/N (none) -> RNCP0603FTD10K0CT-ND; Supplier 1 Price @ Qty (none) -> 0.10; Supplier 1 Unit Price (none) -> 0.10
- TP1: footprint TestPoint:TestPoint_Pad_1.5x1.5mm -> TestPoint:TestPoint_THTPad_1.0x1.0mm_Drill0.5mm
- U3: Mfr (none) -> Microchip Technology; Mfr P/N (none) -> AT42QT1011-TSHR; Supplier 1 (none) -> Digikey; Supplier 1 P/N (none) -> AT42QT1011-TSHRCT-ND; Supplier 1 Price @ Qty (none) -> 0.77000; Supplier 1 Unit Price (none) -> 0.77000
Changed lines of the file:
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@@
+			)
+		)
+		(property "Supplier 1 P/N" "RNCP0603FTD10K0CT-ND"
+			(at 186.69 66.04 0)
+			(effects
+				(font
+					(size 1.27 1.27)
+				)
+				(hide yes)
+			)
+		)
+		(property "Supplier 1 Price @ Qty" "0.10"
+			(at 186.69 66.04 0)
+			(effects
+				(font
+					(size 1.27 1.27)
+				)
+				(hide yes)
+			)
+		)
+		(property "Supplier 1 Unit Price" "0.10"
+			(at 186.69 66.04 0)
+			(effects
+				(font
+					(size 1.27 1.27)
+				)
+				(hide yes)
 			)
 		)
@@
 			)
 		)
+		(property "Supplier_1 P/N" "732-4980-2-ND"
+			(at 80.01 71.12 0)
+			(effects
+				(font
+					(size 1.27 1.27)
+				)
+				(hide yes)
+			)
+		)
+		(property "Supplier_1 Price @ Qty" "0.15000"
+			(at 80.01 71.12 0)
+			(effects
+				(font
+					(size 1.27 1.27)
+				)
+				(hide yes)
+			)
+		)
+		(property "Supplier_1 Unit Price" "0.15000"
+			(at 80.01 71.12 0)
+			(effects
+				(font
+					(size 1.27 1.27)
+				)
+				(hide yes)
+			)
+		)
 		(pin "2"
 		)
@@
 			)
 		)
-		(property "Datasheet" ""
+		(property "Datasheet" "https://ww1.microchip.com/downloads/en/DeviceDoc/40001947A.pdf"
 			(at 147.32 76.2 0)
 			(effects
@@
 			)
 		)
-		(property "Mfr" ""
+		(property "Mfr" "Microchip Technology"
 			(at 147.32 76.2 0)
 			(effects
@@
 			)
 		)
-		(property "Mfr P/N" ""
+		(property "Mfr P/N" "AT42QT1011-TSHR"
 			(at 147.32 76.2 0)
 			(effects
@@
 			)
 		)
-		(property "Supplier 1" ""
+		(property "Supplier 1" "Digikey"
 			(at 147.32 76.2 0)
 			(effects
@@
 			)
 		)
-		(property "Supplier 1 P/N" ""
+		(property "Supplier 1 P/N" "AT42QT1011-TSHRCT-ND"
 			(at 147.32 76.2 0)
 			(effects
@@
 			)
 		)
-		(property "Supplier 1 Unit Price" ""
+		(property "Supplier 1 Unit Price" "0.77000"
 			(at 147.32 76.2 0)
 			(effects
@@
 			)
 		)
-		(property "Supplier 1 Price @ Qty" ""
+		(property "Supplier 1 Price @ Qty" "0.77000"
 			(at 147.32 76.2 0)
 			(effects
@@
 			)
 		)
-		(property "Footprint" "TestPoint:TestPoint_Pad_1.5x1.5mm"
+		(property "Footprint" "TestPoint:TestPoint_THTPad_1.0x1.0mm_Drill0.5mm"
 			(at 196.85 71.12 0)
 			(effects
@@
 		(instances
 			(project ""
+				(path "/f9d381c9-3724-4d31-a5c2-069f1dd9b08c"
+					(reference "TP1")
+					(unit 1)
+				)
 				(path "/f9d381c9-3724-4d31-a5c2-069f1dd9b08c/34dd7306-e107-4822-a0c3-53cc76923bff"
 					(reference "TP1")
@@
 			)
 		)
+		(property "Supplier_1 P/N" "118-CR0603-FX-2000ELFTR-ND"
+			(at 80.01 59.69 0)
+			(effects
+				(font
+					(size 1.27 1.27)
+				)
+				(hide yes)
+			)
+		)
+		(property "Supplier_1 Price @ Qty" "0.10000"
+			(at 80.01 59.69 0)
+			(effects
+				(font
+					(size 1.27 1.27)
+				)
+				(hide yes)
+			)
+		)
+		(property "Supplier_1 Unit Price" "0.10000"
+			(at 80.01 59.69 0)
+			(effects
+				(font
+					(size 1.27 1.27)
+				)
+				(hide yes)
+			)
+		)
 		(pin "2"
 		)
@@
 			)
 		)
+		(property "Supplier_1 P/N" "399-C0402C103K3REC7411TR-ND"
+			(at 173.99 69.85 0)
+			(effects
+				(font
+					(size 1.27 1.27)
+				)
+				(hide yes)
+			)
+		)
+		(property "Supplier_1 Price @ Qty" "0.10000"
+			(at 173.99 69.85 0)
+			(effects
+				(font
+					(size 1.27 1.27)
+				)
+				(hide yes)
+			)
+		)
+		(property "Supplier_1 Unit Price" "0.10000"
+			(at 173.99 69.85 0)
+			(effects
+				(font
+					(size 1.27 1.27)
+				)
+				(hide yes)
+			)
+		)
 		(pin "2"
 		)
@@
 			)
 		)
+		(property "Supplier_1 P/N" "MMBT2222A-FDITR-ND"
+			(at 77.47 86.36 0)
+			(effects
+				(font
+					(size 1.27 1.27)
+				)
+				(hide yes)
+			)
+		)
+		(property "Supplier_1 Price @ Qty" "0.10000"
+			(at 77.47 86.36 0)
+			(effects
+				(font
+					(size 1.27 1.27)
+				)
+				(hide yes)
+			)
+		)
+		(property "Supplier_1 Unit Price" "0.10000"
+			(at 77.47 86.36 0)
+			(effects
+				(font
+					(size 1.27 1.27)
+				)
+				(hide yes)
+			)
+		)
 		(pin "2"
 		)
@@
 			)
 		)
+		(property "Supplier_1 P/N" "399-C0402C103K3REC7411TR-ND"
+			(at 104.14 86.36 0)
+			(effects
+				(font
+					(size 1.27 1.27)
+				)
+				(hide yes)
+			)
+		)
+		(property "Supplier_1 Price @ Qty" "0.10000"
+			(at 104.14 86.36 0)
+			(effects
+				(font
+					(size 1.27 1.27)
+				)
+				(hide yes)
+			)
+		)
+		(property "Supplier_1 Unit Price" "0.10000"
+			(at 104.14 86.36 0)
+			(effects
+				(font
+					(size 1.27 1.27)
+				)
+				(hide yes)
+			)
+		)
 		(pin "1"
 		)
@@
 			)
 		)
-		(property "Supplier 1 P/N" ""
+		(property "Supplier 1 P/N" "A129540CT-ND"
 			(at 64.77 86.36 0)
 			(effects
@@
 			)
 		)
-		(property "Supplier 1 Unit Price" ""
+		(property "Supplier 1 Unit Price" "0.10"
 			(at 64.77 86.36 0)
 			(effects
@@
 			)
 		)
-		(property "Supplier 1 Price @ Qty" ""
+		(property "Supplier 1 Price @ Qty" "0.10"
 			(at 64.77 86.36 0)
 			(effects
