File: power.kicad_sch (KiCad schematic)
At the start: 27 parts, among them Q1 DMP2070UQ-7, SW1 KMR2, U1 MCP73831T-2ACI/OT, U2 AP2112-3.3, X1 JSTPH

Commit message: Updated BOM, created fab outputs
Parts:
- C1, C4, C5, C6, C9: Supplier 1 P/N (none) -> 1276-1096-1-N; Supplier 1 Price @ Qty (none) -> 0.10; Supplier 1 Unit Price (none) -> 0.10
- C10, C11, C12, C2, C3, C7, C8: Supplier 1 P/N (none) -> 311-1446-1-ND; Supplier 1 Price @ Qty (none) -> 0.10; Supplier 1 Unit Price (none) -> 0.10
- CHG1: Supplier 1 P/N (none) -> 3147-B1701UD--20D000414U1930CT-ND; Supplier 1 Price @ Qty (none) -> 0.10; Supplier 1 Unit Price (none) -> 0.10
- D1: Supplier 1 P/N (none) -> MBR120LSFT1GOSCT-ND; Supplier 1 Price @ Qty (none) -> 0.42; Supplier 1 Unit Price (none) -> 0.42
- L1: Supplier 1 P/N (none) -> 587-LSQEA251818T100KCT-ND; Supplier 1 Price @ Qty (none) -> 0.13; Supplier 1 Unit Price (none) -> 0.13
- Q1: Supplier 1 P/N (none) -> 31-DMP2070UQ-7CT-ND; Supplier 1 Price @ Qty (none) -> 0.48; Supplier 1 Unit Price (none) -> 0.48
- R1: Supplier 1 P/N (none) -> MCT0603-1.00K-CFCT-ND; Supplier 1 Price @ Qty (none) -> 0.10; Supplier 1 Unit Price (none) -> 0.10
- R2, R4, R5: Supplier 1 P/N (none) -> RNCP0603FTD10K0CT-ND; Supplier 1 Price @ Qty (none) -> 0.10; Supplier 1 Unit Price (none) -> 0.10
- R3: Supplier 1 P/N (none) -> CR0603-FX-1003ELFTR-ND; Supplier 1 Price @ Qty (none) -> 0.10000; Supplier 1 Unit Price (none) -> 0.10
- R6: Supplier 1 P/N (none) -> CAY16-1003F4LFCT-ND; Supplier 1 Price @ Qty (none) -> 0.10; Supplier 1 Unit Price (none) -> 0.10
- SW1: Supplier 1 P/N (none) -> CKN10285CT-ND; Supplier 1 Price @ Qty (none) -> 0.92; Supplier 1 Unit Price (none) -> 0.92
- U$1: Supplier 1 (none) -> Digikey; Supplier 1 P/N (none) -> ATSAMD51J19A-AUTCT-ND; Supplier 1 Price @ Qty (none) -> 5.68; Supplier 1 Unit Price (none) -> 5.68
- U1: Supplier 1 (none) -> Digikey; Supplier 1 P/N (none) -> MCP73831T-2ATI/OTCT-ND; Supplier 1 Price @ Qty (none) -> 0.76; Supplier 1 Unit Price (none) -> 0.76
- U2: Supplier 1 (none) -> Digikey; Supplier 1 P/N (none) -> AP2112K-3.3TRG1DICT-ND; Supplier 1 Price @ Qty (none) -> 0.35; Supplier 1 Unit Price (none) -> 0.35
- X1: Supplier 1 (none) -> Digikey; Supplier 1 P/N (none) -> 455-S2B-PH-SM4-TBCT-ND; Supplier 1 Price @ Qty (none) -> 0.69000; Supplier 1 Unit Price (none) -> 0.69000
