File: ram.kicad_sch (KiCad schematic)
At the start: 2 parts, among them U4 2MB Flash

Commit message: Updated BOM, created fab outputs
Parts:
- R10: Supplier 1 P/N (none) -> RNCP0603FTD10K0CT-ND; Supplier 1 Price @ Qty (none) -> 0.10; Supplier 1 Unit Price (none) -> 0.10
- U4: Supplier 1 (none) -> Digikey; Supplier 1 P/N (none) -> 1970-GD25Q16ETIGRCT-ND; Supplier 1 Price @ Qty (none) -> 0.74; Supplier 1 Unit Price (none) -> 0.74
Changed lines of the file:
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@@
+			)
+		)
+		(property "Supplier 1 P/N" "1970-GD25Q16ETIGRCT-ND"
+			(at 135.89 116.84 0)
+			(effects
+				(font
+					(size 1.27 1.27)
+				)
+				(hide yes)
+			)
+		)
+		(property "Supplier 1 Price @ Qty" "0.74"
+			(at 135.89 116.84 0)
+			(effects
+				(font
+					(size 1.27 1.27)
+				)
+				(hide yes)
+			)
+		)
+		(property "Supplier 1 Unit Price" "0.74"
+			(at 135.89 116.84 0)
+			(effects
+				(font
+					(size 1.27 1.27)
+				)
+				(hide yes)
+			)
+		)
+		(property "Supplier 1" "Digikey"
+			(at 135.89 116.84 0)
+			(effects
+				(font
+					(size 1.27 1.27)
+				)
+				(hide yes)
 			)
 		)
@@
 			(at 156.21 101.6 0)
 			(effects
+				(font
+					(size 1.27 1.27)
+				)
+				(hide yes)
+			)
+		)
+		(property "Supplier 1 P/N" "RNCP0603FTD10K0CT-ND"
+			(at 156.21 101.6 0)
+			(effects
+				(font
+					(size 1.27 1.27)
+				)
+				(hide yes)
+			)
+		)
+		(property "Supplier 1 Price @ Qty" "0.10"
+			(at 156.21 101.6 0)
+			(effects
+				(font
+					(size 1.27 1.27)
+				)
+				(hide yes)
+			)
+		)
+		(property "Supplier 1 Unit Price" "0.10"
+			(at 156.21 101.6 0)
+			(effects
