File: swd.kicad_sch (KiCad schematic)
At the start: 1 part

Commit message: Updated BOM, created fab outputs
Parts:
- J?: Supplier 1 Price @ Qty (none) -> 1.60000; Supplier 1 Unit Price (none) -> 1.60000; Supplier_1 P/N (none) -> -- mixed values --; Supplier_1 Price @ Qty (none) -> -- mixed values --; Supplier_1 Unit Price (none) -> -- mixed values --
Changed lines of the file:
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@@
 			)
 		)
-		(property "Supplier 1 Unit Price" ""
+		(property "Supplier 1 Unit Price" "1.60000"
 			(at 204.47 134.62 0)
 			(effects
@@
 			)
 		)
-		(property "Supplier 1 Price @ Qty" ""
+		(property "Supplier 1 Price @ Qty" "1.60000"
 			(at 204.47 134.62 0)
 			(effects
@@
 			(at 204.47 134.62 0)
 			(effects
+				(font
+					(size 1.27 1.27)
+				)
+				(hide yes)
+			)
+		)
+		(property "Supplier_1 P/N" "-- mixed values --"
+			(at 204.47 134.62 0)
+			(effects
+				(font
+					(size 1.27 1.27)
+				)
+				(hide yes)
+			)
+		)
+		(property "Supplier_1 Price @ Qty" "-- mixed values --"
+			(at 204.47 134.62 0)
+			(effects
+				(font
+					(size 1.27 1.27)
+				)
+				(hide yes)
+			)
+		)
+		(property "Supplier_1 Unit Price" "-- mixed values --"
+			(at 204.47 134.62 0)
+			(effects
