File: usb.kicad_sch (KiCad schematic)
At the start: 3 parts, among them X2 microUSB 2.0 B

Commit message: Updated BOM, created fab outputs
Parts:
- TP2, TP3: Supplier_1 P/N (none) -> -- mixed values --; Supplier_1 Price @ Qty (none) -> -- mixed values --; Supplier_1 Unit Price (none) -> -- mixed values --
- X2: Mfr P/N 10118194-0001LF -> 10103594-0001LF; Supplier 1 (none) -> Digikey; Supplier 1 P/N (none) -> 609-4050-2-ND; Supplier 1 Price @ Qty (none) -> 0.84000; Supplier 1 Unit Price (none) -> 0.84000
Changed lines of the file:
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@@
 			)
 		)
-		(property "Mfr P/N" "10118194-0001LF"
+		(property "Mfr P/N" "10103594-0001LF"
 			(at 133.35 97.79 0)
 			(effects
@@
 		)
 		(property "Supplier_2 Price @ Qty" ""
+			(at 133.35 97.79 0)
+			(effects
+				(font
+					(size 1.27 1.27)
+				)
+				(hide yes)
+			)
+		)
+		(property "Supplier 1 P/N" "609-4050-2-ND"
+			(at 133.35 97.79 0)
+			(effects
+				(font
+					(size 1.27 1.27)
+				)
+				(hide yes)
+			)
+		)
+		(property "Supplier 1 Price @ Qty" "0.84000"
+			(at 133.35 97.79 0)
+			(effects
+				(font
+					(size 1.27 1.27)
+				)
+				(hide yes)
+			)
+		)
+		(property "Supplier 1 Unit Price" "0.84000"
+			(at 133.35 97.79 0)
+			(effects
+				(font
+					(size 1.27 1.27)
+				)
+				(hide yes)
+			)
+		)
+		(property "Supplier 1" "Digikey"
 			(at 133.35 97.79 0)
 			(effects
@@
 			)
 		)
-		(property "Supplier_1 P/N" ""
-			(at 160.02 105.41 0)
-			(effects
-				(font
-					(size 1.27 1.27)
-				)
-				(hide yes)
-			)
-		)
-		(property "Supplier_1 Unit Price" ""
-			(at 160.02 105.41 0)
-			(effects
-				(font
-					(size 1.27 1.27)
-				)
-				(hide yes)
-			)
-		)
-		(property "Supplier_1 Price @ Qty" ""
+		(property "Supplier_1 P/N" "-- mixed values --"
+			(at 160.02 105.41 0)
+			(effects
+				(font
+					(size 1.27 1.27)
+				)
+				(hide yes)
+			)
+		)
+		(property "Supplier_1 Unit Price" "-- mixed values --"
+			(at 160.02 105.41 0)
+			(effects
+				(font
+					(size 1.27 1.27)
+				)
+				(hide yes)
+			)
+		)
+		(property "Supplier_1 Price @ Qty" "-- mixed values --"
 			(at 160.02 105.41 0)
 			(effects
@@
 			)
 		)
-		(property "Supplier_1 P/N" ""
-			(at 160.02 92.71 0)
-			(effects
-				(font
-					(size 1.27 1.27)
-				)
-				(hide yes)
-			)
-		)
-		(property "Supplier_1 Unit Price" ""
-			(at 160.02 92.71 0)
-			(effects
-				(font
-					(size 1.27 1.27)
-				)
-				(hide yes)
-			)
-		)
-		(property "Supplier_1 Price @ Qty" ""
-			(at 160.02 92.71 0)
-			(effects
+		(property "Supplier_1 P/N" "-- mixed values --"
+			(at 160.02 92.71 0)
+			(effects
+				(font
+					(size 1.27 1.27)
+				)
+				(hide yes)
+			)
+		)
+		(property "Supplier_1 Unit Price" "-- mixed values --"
+			(at 160.02 92.71 0)
+			(effects
+				(font
+					(size 1.27 1.27)
+				)
+				(hide yes)
+			)
+		)
+		(property "Supplier_1 Price @ Qty" "-- mixed values --"
+			(at 160.02 92.71 0)
+			(effects
