File: wifi.kicad_sch (KiCad schematic)
At the start: 5 parts, among them J3 Conn_01x12_Socket

Commit message: Updated BOM, created fab outputs
Parts:
- J3: Supplier_1 P/N (none) -> S6100-ND; Supplier_1 Price @ Qty (none) -> 0.97000; Supplier_1 Unit Price (none) -> 0.97000
- R23, R24, R25, R26: Supplier 1 P/N (none) -> 311-0.0GRTR-ND; Supplier 1 Price @ Qty (none) -> 0.00900; Supplier 1 Unit Price (none) -> 0.10
Changed lines of the file:
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@@
 			)
 		)
-		(property "Supplier 1 P/N" ""
+		(property "Supplier 1 P/N" "311-0.0GRTR-ND"
 			(at 127 101.6 0)
 			(effects
@@
 			)
 		)
-		(property "Supplier 1 Unit Price" ""
+		(property "Supplier 1 Unit Price" "0.10"
 			(at 127 101.6 0)
 			(effects
@@
 			)
 		)
-		(property "Supplier 1 Price @ Qty" ""
+		(property "Supplier 1 Price @ Qty" "0.00900"
 			(at 127 101.6 0)
 			(effects
@@
 			)
 		)
-		(property "Supplier 1 P/N" ""
-			(at 127 96.52 0)
-			(effects
-				(font
-					(size 1.27 1.27)
-				)
-				(hide yes)
-			)
-		)
-		(property "Supplier 1 Unit Price" ""
-			(at 127 96.52 0)
-			(effects
-				(font
-					(size 1.27 1.27)
-				)
-				(hide yes)
-			)
-		)
-		(property "Supplier 1 Price @ Qty" ""
+		(property "Supplier 1 P/N" "311-0.0GRTR-ND"
+			(at 127 96.52 0)
+			(effects
+				(font
+					(size 1.27 1.27)
+				)
+				(hide yes)
+			)
+		)
+		(property "Supplier 1 Unit Price" "0.10"
+			(at 127 96.52 0)
+			(effects
+				(font
+					(size 1.27 1.27)
+				)
+				(hide yes)
+			)
+		)
+		(property "Supplier 1 Price @ Qty" "0.00900"
 			(at 127 96.52 0)
 			(effects
@@
 			)
 		)
+		(property "Supplier_1 P/N" "S6100-ND"
+			(at 99.06 99.06 0)
+			(effects
+				(font
+					(size 1.27 1.27)
+				)
+				(hide yes)
+			)
+		)
+		(property "Supplier_1 Price @ Qty" "0.97000"
+			(at 99.06 99.06 0)
+			(effects
+				(font
+					(size 1.27 1.27)
+				)
+				(hide yes)
+			)
+		)
+		(property "Supplier_1 Unit Price" "0.97000"
+			(at 99.06 99.06 0)
+			(effects
+				(font
+					(size 1.27 1.27)
+				)
+				(hide yes)
+			)
+		)
 		(pin "9"
 		)
@@
 			)
 		)
-		(property "Supplier 1 P/N" ""
-			(at 127 99.06 0)
-			(effects
-				(font
-					(size 1.27 1.27)
-				)
-				(hide yes)
-			)
-		)
-		(property "Supplier 1 Unit Price" ""
-			(at 127 99.06 0)
-			(effects
-				(font
-					(size 1.27 1.27)
-				)
-				(hide yes)
-			)
-		)
-		(property "Supplier 1 Price @ Qty" ""
+		(property "Supplier 1 P/N" "311-0.0GRTR-ND"
+			(at 127 99.06 0)
+			(effects
+				(font
+					(size 1.27 1.27)
+				)
+				(hide yes)
+			)
+		)
+		(property "Supplier 1 Unit Price" "0.10"
+			(at 127 99.06 0)
+			(effects
+				(font
+					(size 1.27 1.27)
+				)
+				(hide yes)
+			)
+		)
+		(property "Supplier 1 Price @ Qty" "0.00900"
 			(at 127 99.06 0)
 			(effects
@@
 			)
 		)
-		(property "Supplier 1 P/N" ""
-			(at 127 93.98 0)
-			(effects
-				(font
-					(size 1.27 1.27)
-				)
-				(hide yes)
-			)
-		)
-		(property "Supplier 1 Unit Price" ""
-			(at 127 93.98 0)
-			(effects
-				(font
-					(size 1.27 1.27)
-				)
-				(hide yes)
-			)
-		)
-		(property "Supplier 1 Price @ Qty" ""
-			(at 127 93.98 0)
-			(effects
+		(property "Supplier 1 P/N" "311-0.0GRTR-ND"
+			(at 127 93.98 0)
+			(effects
+				(font
+					(size 1.27 1.27)
+				)
+				(hide yes)
+			)
+		)
+		(property "Supplier 1 Unit Price" "0.10"
+			(at 127 93.98 0)
+			(effects
+				(font
+					(size 1.27 1.27)
+				)
+				(hide yes)
+			)
+		)
+		(property "Supplier 1 Price @ Qty" "0.00900"
+			(at 127 93.98 0)
+			(effects
