File: temp.kicad_sch (KiCad schematic)
At the start: 6 parts, among them U5 MCP9808-E_MS

Commit message: Updated BOM, created fab outputs
Parts:
- C17: Supplier 1 P/N (none) -> 311-1446-1-ND; Supplier 1 Price @ Qty (none) -> 0.10; Supplier 1 Unit Price (none) -> 0.10
- R27, R28: Supplier 1 P/N (none) -> 311-0.0GRTR-ND; Supplier 1 Price @ Qty (none) -> 0.00900; Supplier 1 Unit Price (none) -> 0.10
- R29, R30: Supplier 1 P/N (none) -> RNCP0603FTD10K0CT-ND; Supplier 1 Price @ Qty (none) -> 0.10; Supplier 1 Unit Price (none) -> 0.10
- U5: Supplier_1 P/N (none) -> MCP9808-E/MS-ND; Supplier_1 Price @ Qty (none) -> 1.40; Supplier_1 Unit Price (none) -> 1.40
Changed lines of the file:
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@@
+			)
+		)
+		(property "Supplier 1 P/N" "311-1446-1-ND"
+			(at 187.96 95.25 0)
+			(effects
+				(font
+					(size 1.27 1.27)
+				)
+				(hide yes)
+			)
+		)
+		(property "Supplier 1 Price @ Qty" "0.10"
+			(at 187.96 95.25 0)
+			(effects
+				(font
+					(size 1.27 1.27)
+				)
+				(hide yes)
+			)
+		)
+		(property "Supplier 1 Unit Price" "0.10"
+			(at 187.96 95.25 0)
+			(effects
+				(font
+					(size 1.27 1.27)
+				)
+				(hide yes)
 			)
 		)
@@
 			)
 		)
+		(property "Supplier_1 P/N" "MCP9808-E/MS-ND"
+			(at 140.97 106.68 0)
+			(effects
+				(font
+					(size 1.27 1.27)
+				)
+				(hide yes)
+			)
+		)
+		(property "Supplier_1 Price @ Qty" "1.40"
+			(at 140.97 106.68 0)
+			(effects
+				(font
+					(size 1.27 1.27)
+				)
+				(hide yes)
+			)
+		)
+		(property "Supplier_1 Unit Price" "1.40"
+			(at 140.97 106.68 0)
+			(effects
+				(font
+					(size 1.27 1.27)
+				)
+				(hide yes)
+			)
+		)
 		(pin "6"
 		)
@@
 			)
 		)
-		(property "Supplier 1 P/N" ""
-			(at 104.14 99.06 0)
-			(effects
-				(font
-					(size 1.27 1.27)
-				)
-				(hide yes)
-			)
-		)
-		(property "Supplier 1 Unit Price" ""
-			(at 104.14 99.06 0)
-			(effects
-				(font
-					(size 1.27 1.27)
-				)
-				(hide yes)
-			)
-		)
-		(property "Supplier 1 Price @ Qty" ""
+		(property "Supplier 1 P/N" "311-0.0GRTR-ND"
+			(at 104.14 99.06 0)
+			(effects
+				(font
+					(size 1.27 1.27)
+				)
+				(hide yes)
+			)
+		)
+		(property "Supplier 1 Unit Price" "0.10"
+			(at 104.14 99.06 0)
+			(effects
+				(font
+					(size 1.27 1.27)
+				)
+				(hide yes)
+			)
+		)
+		(property "Supplier 1 Price @ Qty" "0.00900"
 			(at 104.14 99.06 0)
 			(effects
@@
 			)
 		)
-		(property "Supplier 1 P/N" ""
-			(at 110.49 85.09 0)
-			(effects
-				(font
-					(size 1.27 1.27)
-				)
-				(hide yes)
-			)
-		)
-		(property "Supplier 1 Unit Price" ""
-			(at 110.49 85.09 0)
-			(effects
-				(font
-					(size 1.27 1.27)
-				)
-				(hide yes)
-			)
-		)
-		(property "Supplier 1 Price @ Qty" ""
+		(property "Supplier 1 P/N" "RNCP0603FTD10K0CT-ND"
+			(at 110.49 85.09 0)
+			(effects
+				(font
+					(size 1.27 1.27)
+				)
+				(hide yes)
+			)
+		)
+		(property "Supplier 1 Unit Price" "0.10"
+			(at 110.49 85.09 0)
+			(effects
+				(font
+					(size 1.27 1.27)
+				)
+				(hide yes)
+			)
+		)
+		(property "Supplier 1 Price @ Qty" "0.10"
 			(at 110.49 85.09 0)
 			(effects
@@
 			)
 		)
-		(property "Supplier 1 P/N" ""
-			(at 119.38 91.44 0)
-			(effects
-				(font
-					(size 1.27 1.27)
-				)
-				(hide yes)
-			)
-		)
-		(property "Supplier 1 Unit Price" ""
-			(at 119.38 91.44 0)
-			(effects
-				(font
-					(size 1.27 1.27)
-				)
-				(hide yes)
-			)
-		)
-		(property "Supplier 1 Price @ Qty" ""
+		(property "Supplier 1 P/N" "RNCP0603FTD10K0CT-ND"
+			(at 119.38 91.44 0)
+			(effects
+				(font
+					(size 1.27 1.27)
+				)
+				(hide yes)
+			)
+		)
+		(property "Supplier 1 Unit Price" "0.10"
+			(at 119.38 91.44 0)
+			(effects
+				(font
+					(size 1.27 1.27)
+				)
+				(hide yes)
+			)
+		)
+		(property "Supplier 1 Price @ Qty" "0.10"
 			(at 119.38 91.44 0)
 			(effects
@@
 			)
 		)
-		(property "Supplier 1 P/N" ""
-			(at 104.14 101.6 0)
-			(effects
-				(font
-					(size 1.27 1.27)
-				)
-				(hide yes)
-			)
-		)
-		(property "Supplier 1 Unit Price" ""
-			(at 104.14 101.6 0)
-			(effects
-				(font
-					(size 1.27 1.27)
-				)
-				(hide yes)
-			)
-		)
-		(property "Supplier 1 Price @ Qty" ""
-			(at 104.14 101.6 0)
-			(effects
+		(property "Supplier 1 P/N" "311-0.0GRTR-ND"
+			(at 104.14 101.6 0)
+			(effects
+				(font
+					(size 1.27 1.27)
+				)
+				(hide yes)
+			)
+		)
+		(property "Supplier 1 Unit Price" "0.10"
+			(at 104.14 101.6 0)
+			(effects
+				(font
+					(size 1.27 1.27)
+				)
+				(hide yes)
+			)
+		)
+		(property "Supplier 1 Price @ Qty" "0.00900"
+			(at 104.14 101.6 0)
+			(effects

Commit message: Final project submission
Connections:
- net A0 is gone; now on net GND: U5.7 (A0)
- net A1 is gone; now on net GND: U5.6 (A1)
- net A2 is gone; now on net GND: U5.5 (A2)
- no-connect marks 4 -> 1
Other:
- note added: "A0, A1, A2 for setting I2C address. GND: default 0x18 https://learn.adafruit.com/adafruit-mcp9808-precision-i2c-temperature-sensor-guide/pinouts"
- note removed: "A0, A1, A2 for setting I2C address. Unconnected: default 0x18 https://learn.adafruit.com/adafruit-mcp9808-precision-i2c-temperature-sensor-guide/pinouts"
Changed lines of the file:
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@@
+	)
+	(junction
+		(at 175.26 110.49)
+		(diameter 0)
+		(color 0 0 0 0)
 	)
 	(junction
@@
 		(color 0 0 0 0)
 	)
-	(no_connect
-		(at 175.26 110.49)
-	)
-	(no_connect
+	(junction
 		(at 175.26 113.03)
+		(diameter 0)
+		(color 0 0 0 0)
 	)
 	(no_connect
 		(at 113.03 106.68)
-	)
-	(no_connect
-		(at 175.26 107.95)
 	)
 	(bus_entry
@@
 	(wire
 		(pts
+			(xy 175.26 115.57) (xy 175.26 113.03)
+		)
+		(stroke
+			(width 0)
+			(type default)
+		)
+	)
+	(wire
+		(pts
 			(xy 217.17 100.33) (xy 217.17 91.44)
 		)
@@
 	(wire
 		(pts
+			(xy 175.26 107.95) (xy 175.26 110.49)
+		)
+		(stroke
+			(width 0)
+			(type default)
+		)
+	)
+	(wire
+		(pts
 			(xy 100.33 99.06) (xy 95.25 99.06)
 		)
@@
 	(wire
 		(pts
+			(xy 175.26 110.49) (xy 175.26 113.03)
+		)
+		(stroke
+			(width 0)
+			(type default)
+		)
+	)
+	(wire
+		(pts
 			(xy 175.26 110.49) (xy 162.56 110.49)
 		)
@@
 		)
 	)
-	(text "A0, A1, A2 for setting I2C address.\nUnconnected: default 0x18\nhttps://learn.adafruit.com/adafruit-mcp9808-precision-i2c-temperature-sensor-guide/pinouts"
+	(text "A0, A1, A2 for setting I2C address.\nGND: default 0x18\nhttps://learn.adafruit.com/adafruit-mcp9808-precision-i2c-temperature-sensor-guide/pinouts"
 		(exclude_from_sim no)
 		(at 158.75 120.65 0)
@@
 		(fields_autoplaced yes)
 		(effects
+			(font
+				(size 1.27 1.27)
+			)
+			(justify left bottom)
+		)
+	)
+	(label "GND"
+		(at 175.26 115.57 0)
+		(fields_autoplaced yes)
+		(effects
